Commit message: Parte 2: chasis con dos ruedas y casters

File: src/mi_robot_diferencial/urdf/mi_robot.urdf.xacro (robot description, xacro)
@@ -1,17 +1,17 @@
 <?xml version="1.0"?>
 <robot name="mi_robot" xmlns:xacro="http://www.ros.org/wiki/xacro">
+  <!-- ===== Parámetros: se cambian aquí y se actualizan en todo el archivo ===== -->
+  <xacro:property name="rueda_radio" value="0.05"/>
+  <xacro:property name="rueda_ancho" value="0.03"/>
+  <xacro:property name="separacion_ruedas" value="0.25"/>
+  <xacro:property name="caster_radio" value="0.01"/>
+  <!-- ===== Chasis ===== -->
   <link name="base_link">
     <visual>
-      <geometry>
-        <box size="0.3 0.2 0.1"/>
-      </geometry>
-      <material name="azul">
-        <color rgba="0.2 0.4 0.8 1"/>
-      </material>
+      <geometry><box size="0.3 0.2 0.1"/></geometry>
+      <material name="azul"><color rgba="0.2 0.4 0.8 1"/></material>
     </visual>
     <collision>
-      <geometry>
-        <box size="0.3 0.2 0.1"/>
-      </geometry>
+      <geometry><box size="0.3 0.2 0.1"/></geometry>
     </collision>
     <inertial>
@@ -20,3 +20,57 @@
     </inertial>
   </link>
+  <!-- ===== Plantilla de rueda (se usa dos veces: izquierda y derecha) ===== -->
+  <xacro:macro name="rueda" params="prefijo y_signo">
+    <link name="rueda_${prefijo}">
+      <visual>
+        <geometry><cylinder radius="${rueda_radio}" length="${rueda_ancho}"/></geometry>
+        <material name="negro"><color rgba="0.1 0.1 0.1 1"/></material>
+      </visual>
+      <collision>
+        <geometry><cylinder radius="${rueda_radio}" length="${rueda_ancho}"/></geometry>
+      </collision>
+      <inertial>
+        <mass value="0.1"/>
+        <inertia ixx="0.0005" ixy="0.0" ixz="0.0" iyy="0.0005" iyz="0.0" izz="0.0005"/>
+      </inertial>
+    </link>
+    <joint name="joint_rueda_${prefijo}" type="continuous">
+      <parent link="base_link"/>
+      <child link="rueda_${prefijo}"/>
+      <!-- rpy = -90°: el eje de la rueda apunta a +y, así un giro positivo hace avanzar en +x -->
+      <origin xyz="0 ${y_signo * separacion_ruedas/2} -0.02" rpy="-1.5708 0 0"/>
+      <axis xyz="0 0 1"/>
+    </joint>
+  </xacro:macro>
+  <xacro:rueda prefijo="izq" y_signo="1"/>
+  <xacro:rueda prefijo="der" y_signo="-1"/>
+  <!-- ===== Casters: apoyos adelante y atrás para que el chasis no se incline ===== -->
+  <xacro:macro name="caster" params="prefijo x">
+    <link name="caster_${prefijo}">
+      <visual>
+        <geometry><sphere radius="${caster_radio}"/></geometry>
+        <material name="gris"><color rgba="0.6 0.6 0.6 1"/></material>
+      </visual>
+      <collision>
+        <geometry><sphere radius="${caster_radio}"/></geometry>
+      </collision>
+      <inertial>
+        <mass value="0.01"/>
+        <inertia ixx="1e-6" ixy="0.0" ixz="0.0" iyy="1e-6" iyz="0.0" izz="1e-6"/>
+      </inertial>
+    </link>
+    <joint name="joint_caster_${prefijo}" type="fixed">
+      <parent link="base_link"/>
+      <child link="caster_${prefijo}"/>
+      <!-- El fondo de la esfera queda a la misma altura que el fondo de las ruedas -->
+      <origin xyz="${x} 0 ${-0.02 - rueda_radio + caster_radio}" rpy="0 0 0"/>
+    </joint>
+    <!-- Sin fricción: la esfera se desliza y no frena al robot -->
+    <gazebo reference="caster_${prefijo}">
+      <mu1>0.0</mu1>
+      <mu2>0.0</mu2>
+    </gazebo>
+  </xacro:macro>
+  <xacro:caster prefijo="del" x="0.12"/>
+  <xacro:caster prefijo="tra" x="-0.12"/>
 </robot>

Commit message: Parte 5: LiDAR y camara en el Xacro

File: src/mi_robot_diferencial/urdf/mi_robot.urdf.xacro (robot description, xacro)
@@ -74,4 +74,100 @@
   <xacro:caster prefijo="del" x="0.12"/>
   <xacro:caster prefijo="tra" x="-0.12"/>
+  <!-- ===== LiDAR ===== -->
+  <link name="lidar_link">
+    <visual>
+      <geometry><cylinder radius="0.035" length="0.04"/></geometry>
+      <material name="rojo"><color rgba="0.8 0.1 0.1 1"/></material>
+    </visual>
+    <collision>
+      <geometry><cylinder radius="0.035" length="0.04"/></geometry>
+    </collision>
+    <inertial>
+      <mass value="0.17"/>
+      <inertia ixx="0.0001" ixy="0" ixz="0" iyy="0.0001" iyz="0" izz="0.0001"/>
+    </inertial>
+  </link>
+  <joint name="joint_lidar" type="fixed">
+    <parent link="base_link"/>
+    <child link="lidar_link"/>
+    <!-- Centrado encima del chasis: ve 360° sin que el propio robot le tape los rayos -->
+    <origin xyz="0 0 0.07" rpy="0 0 0"/>
+  </joint>
+  <gazebo reference="lidar_link">
+    <sensor name="lidar" type="gpu_lidar">
+      <gz_frame_id>lidar_link</gz_frame_id>   <!-- frame que aparece en el mensaje /scan -->
+      <topic>scan</topic>
+      <update_rate>10</update_rate>          <!-- 10 Hz -->
+      <always_on>true</always_on>
+      <visualize>true</visualize>            <!-- dibuja los rayos en Gazebo -->
+      <lidar>
+        <scan>
+          <horizontal>
+            <samples>360</samples>           <!-- 360 muestras = 1 por grado -->
+            <resolution>1</resolution>
+            <min_angle>-3.14159</min_angle>  <!-- FOV de 360° -->
+            <max_angle>3.14159</max_angle>
+          </horizontal>
+        </scan>
+        <range>
+          <min>0.15</min>                    <!-- rango mínimo [m] -->
+          <max>12.0</max>                    <!-- rango máximo [m] -->
+          <resolution>0.01</resolution>
+        </range>
+        <noise>                              <!-- ruido de medición, como un sensor real -->
+          <type>gaussian</type>
+          <mean>0.0</mean>
+          <stddev>0.01</stddev>
+        </noise>
+      </lidar>
+    </sensor>
+  </gazebo>
+  <!-- ===== Cámara ===== -->
+  <link name="camera_link">
+    <visual>
+      <geometry><box size="0.02 0.05 0.03"/></geometry>
+      <material name="verde"><color rgba="0.1 0.7 0.1 1"/></material>
+    </visual>
+    <collision>
+      <geometry><box size="0.02 0.05 0.03"/></geometry>
+    </collision>
+    <inertial>
+      <mass value="0.03"/>
+      <inertia ixx="0.00001" ixy="0" ixz="0" iyy="0.00001" iyz="0" izz="0.00001"/>
+    </inertial>
+  </link>
+  <joint name="joint_camara" type="fixed">
+    <parent link="base_link"/>
+    <child link="camera_link"/>
+    <!-- En la cara frontal del chasis, mirando hacia adelante (+x) -->
+    <origin xyz="0.16 0 0.02" rpy="0 0 0"/>
+  </joint>
+  <!-- Frame óptico: las imágenes usan z hacia adelante, x a la derecha, y hacia abajo -->
+  <link name="camera_optical_link"/>
+  <joint name="joint_camara_optica" type="fixed">
+    <parent link="camera_link"/>
+    <child link="camera_optical_link"/>
+    <origin xyz="0 0 0" rpy="-1.5708 0 -1.5708"/>
+  </joint>
+  <gazebo reference="camera_link">
+    <sensor name="camara" type="camera">
+      <gz_frame_id>camera_optical_link</gz_frame_id>
+      <topic>image_raw</topic>               <!-- camera_info sale solo en /camera_info -->
+      <update_rate>30</update_rate>          <!-- 30 FPS -->
+      <always_on>true</always_on>
+      <camera>
+        <horizontal_fov>1.0856</horizontal_fov>   <!-- 62.2° -->
+        <image>
+          <width>640</width>
+          <height>480</height>
+          <format>R8G8B8</format>
+        </image>
+        <clip>
+          <near>0.05</near>
+          <far>20.0</far>
+        </clip>
+      </camera>
+    </sensor>
+  </gazebo>
   <!-- ===== Plugins de Gazebo ===== -->
   <gazebo>

Commit message: Inercias calculadas con formulas de solidos y friccion en ruedas

File: src/mi_robot_diferencial/urdf/mi_robot.urdf.xacro (robot description, xacro)
@@ -2,21 +2,49 @@
 <robot name="mi_robot" xmlns:xacro="http://www.ros.org/wiki/xacro">
   <!-- ===== Parámetros: se cambian aquí y se actualizan en todo el archivo ===== -->
+  <xacro:property name="chasis_largo" value="0.30"/>
+  <xacro:property name="chasis_ancho" value="0.20"/>
+  <xacro:property name="chasis_alto" value="0.10"/>
+  <xacro:property name="chasis_masa" value="1.5"/>
   <xacro:property name="rueda_radio" value="0.05"/>
   <xacro:property name="rueda_ancho" value="0.03"/>
+  <xacro:property name="rueda_masa" value="0.2"/>
   <xacro:property name="separacion_ruedas" value="0.25"/>
   <xacro:property name="caster_radio" value="0.01"/>
+  <xacro:property name="caster_masa" value="0.02"/>
+  <!-- ===== Fórmulas de inercia de sólidos ===== -->
+  <xacro:macro name="inercia_caja" params="m x y z">
+    <inertial>
+      <mass value="${m}"/>
+      <inertia ixx="${m*(y*y+z*z)/12}" ixy="0" ixz="0"
+               iyy="${m*(x*x+z*z)/12}" iyz="0"
+               izz="${m*(x*x+y*y)/12}"/>
+    </inertial>
+  </xacro:macro>
+  <xacro:macro name="inercia_cilindro" params="m r h">
+    <inertial>
+      <mass value="${m}"/>
+      <inertia ixx="${m*(3*r*r+h*h)/12}" ixy="0" ixz="0"
+               iyy="${m*(3*r*r+h*h)/12}" iyz="0"
+               izz="${m*r*r/2}"/>
+    </inertial>
+  </xacro:macro>
+  <xacro:macro name="inercia_esfera" params="m r">
+    <inertial>
+      <mass value="${m}"/>
+      <inertia ixx="${2*m*r*r/5}" ixy="0" ixz="0"
+               iyy="${2*m*r*r/5}" iyz="0"
+               izz="${2*m*r*r/5}"/>
+    </inertial>
+  </xacro:macro>
   <!-- ===== Chasis ===== -->
   <link name="base_link">
     <visual>
-      <geometry><box size="0.3 0.2 0.1"/></geometry>
+      <geometry><box size="${chasis_largo} ${chasis_ancho} ${chasis_alto}"/></geometry>
       <material name="azul"><color rgba="0.2 0.4 0.8 1"/></material>
     </visual>
     <collision>
-      <geometry><box size="0.3 0.2 0.1"/></geometry>
+      <geometry><box size="${chasis_largo} ${chasis_ancho} ${chasis_alto}"/></geometry>
     </collision>
-    <inertial>
-      <mass value="1.0"/>
-      <inertia ixx="0.01" ixy="0.0" ixz="0.0" iyy="0.01" iyz="0.0" izz="0.01"/>
-    </inertial>
+    <xacro:inercia_caja m="${chasis_masa}" x="${chasis_largo}" y="${chasis_ancho}" z="${chasis_alto}"/>
   </link>
   <!-- ===== Plantilla de rueda (se usa dos veces: izquierda y derecha) ===== -->
@@ -30,8 +58,5 @@
         <geometry><cylinder radius="${rueda_radio}" length="${rueda_ancho}"/></geometry>
       </collision>
-      <inertial>
-        <mass value="0.1"/>
-        <inertia ixx="0.0005" ixy="0.0" ixz="0.0" iyy="0.0005" iyz="0.0" izz="0.0005"/>
-      </inertial>
+      <xacro:inercia_cilindro m="${rueda_masa}" r="${rueda_radio}" h="${rueda_ancho}"/>
     </link>
     <joint name="joint_rueda_${prefijo}" type="continuous">
@@ -42,4 +67,9 @@
       <axis xyz="0 0 1"/>
     </joint>
+    <!-- Fricción alta: la rueda agarra el piso y no patina -->
+    <gazebo reference="rueda_${prefijo}">
+      <mu1>1.0</mu1>
+      <mu2>1.0</mu2>
+    </gazebo>
   </xacro:macro>
   <xacro:rueda prefijo="izq" y_signo="1"/>
@@ -55,8 +85,5 @@
         <geometry><sphere radius="${caster_radio}"/></geometry>
       </collision>
-      <inertial>
-        <mass value="0.01"/>
-        <inertia ixx="1e-6" ixy="0.0" ixz="0.0" iyy="1e-6" iyz="0.0" izz="1e-6"/>
-      </inertial>
+      <xacro:inercia_esfera m="${caster_masa}" r="${caster_radio}"/>
     </link>
     <joint name="joint_caster_${prefijo}" type="fixed">
@@ -83,8 +110,5 @@
       <geometry><cylinder radius="0.035" length="0.04"/></geometry>
     </collision>
-    <inertial>
-      <mass value="0.17"/>
-      <inertia ixx="0.0001" ixy="0" ixz="0" iyy="0.0001" iyz="0" izz="0.0001"/>
-    </inertial>
+    <xacro:inercia_cilindro m="0.17" r="0.035" h="0.04"/>
   </link>
   <joint name="joint_lidar" type="fixed">
@@ -100,5 +124,5 @@
       <update_rate>10</update_rate>          <!-- 10 Hz -->
       <always_on>true</always_on>
-      <visualize>true</visualize>            <!-- dibuja los rayos en Gazebo -->
+      <visualize>true</visualize>
       <lidar>
         <scan>
@@ -132,8 +156,5 @@
       <geometry><box size="0.02 0.05 0.03"/></geometry>
     </collision>
-    <inertial>
-      <mass value="0.03"/>
-      <inertia ixx="0.00001" ixy="0" ixz="0" iyy="0.00001" iyz="0" izz="0.00001"/>
-    </inertial>
+    <xacro:inercia_caja m="0.03" x="0.02" y="0.05" z="0.03"/>
   </link>
   <joint name="joint_camara" type="fixed">

Commit message: Casters con tamano real (Pololu 1 pulgada) y carcasa visible

File: src/mi_robot_diferencial/urdf/mi_robot.urdf.xacro (robot description, xacro)
@@ -10,6 +10,6 @@
   <xacro:property name="rueda_masa" value="0.2"/>
   <xacro:property name="separacion_ruedas" value="0.25"/>
-  <xacro:property name="caster_radio" value="0.01"/>
-  <xacro:property name="caster_masa" value="0.02"/>
+  <xacro:property name="caster_radio" value="0.0127"/>
+  <xacro:property name="caster_masa" value="0.0185"/>
   <!-- ===== Fórmulas de inercia de sólidos ===== -->
   <xacro:macro name="inercia_caja" params="m x y z">
@@ -80,5 +80,10 @@
       <visual>
         <geometry><sphere radius="${caster_radio}"/></geometry>
-        <material name="gris"><color rgba="0.6 0.6 0.6 1"/></material>
+        <material name="blanco"><color rgba="0.9 0.9 0.9 1"/></material>
+      </visual>
+      <visual>
+        <origin xyz="0 0 0.01" rpy="0 0 0"/>
+        <geometry><cylinder radius="0.017" length="0.02"/></geometry>
+        <material name="negro"><color rgba="0.1 0.1 0.1 1"/></material>
       </visual>
       <collision>
